File: Lab5_Mechatronics/Colpitts_Simulatable/Colpitts_Simulatable.kicad_sch (KiCad schematic)
At the start: 12 parts, among them Q1 2N3904

Commit message: added simulation models
Parts:
- added C5, C6, C7: 0.1u, symbol Device:C
- added L2: 10u, symbol Device:L_Trim
- added Q2, Q3: 2N3904, Package_TO_SOT_THT:TO-92_Inline, symbol Transistor_BJT:2N3904
- added R10, R5, R6, R7: 1k, symbol Device:R_US
- added R8, R9: 22k, symbol Device:R_US
- added V3, V4, V5, V6: 5, symbol Simulation_SPICE:VDC
Connections:
- net GND: now also Q3.1 (E), R6.2, R7.2, R9.2, V3.2, V4.2, V5.2, V6.2
- new net: C7.2, Q3.2 (B), R8.2, R9.1
- new net: Q3.3 (C), R10.2
- new net: C5.1, L2.1, V4.1
- new net: C5.2, C6.1, C7.1, Q2.1 (E), R7.1
- new net: C6.2, L2.2, Q2.3 (C)
- new net: Q2.2 (B), R5.2, R6.1
- new net: R5.1, V3.1
- new net: R8.1, V5.1
- new net: R10.1, V6.1
Other:
- note added: ".tran 10n 1m"
- note removed: ".tran 10u 100m"
