File: Lab5_Mechatronics/Lab5_Mechatronics.kicad_sch (KiCad schematic)
At the start: 22 parts, among them Q1 2N3904, Q2 2N3904, Q3 2N3904

Commit message: replaced 100k with 1Meg
Parts:
- R1: value 100k -> 1Meg
Changed lines of the file:
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@@
       (effects (font (size 1.27 1.27)) (justify left))
     )
-    (property "Value" "100k" (at 71.12 34.29 0)
+    (property "Value" "1Meg" (at 71.12 34.29 0)
       (effects (font (size 1.27 1.27)) (justify left))
     )
