File: Lab6_Mechatronics/Lab6_Mechatronics/Lab6_Mechatronics.kicad_sch (KiCad schematic)
At the start: 7 parts, among them U1 TMP36xS

Commit message: minor fix
Connections:
- net ADC_GPI renamed GPI_ADC
Changed lines of the file:
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@@
     (effects (font (size 1.27 1.27) (color 255 255 255 1)) (justify left bottom))
   )
-  (label "ADC_GPI" (at 163.83 52.07 0) (fields_autoplaced)
+  (label "GPI_ADC" (at 163.83 52.07 0) (fields_autoplaced)
     (effects (font (size 1.27 1.27)) (justify left bottom))
   )
